Commit message: fix(urdf): add base_footprint link and joint for RViz2 frame resolution

File: simulation/urdf/advika.urdf (robot description, URDF)
Before this commit: robot advika, 12 links, 11 joints
Links:
- added link base_footprint
Joints:
- added joint base_footprint_joint: type fixed, parent base_footprint, child base_link, origin xyz=0 0 0.0 rpy=0 0 0

File: src/advika_description/urdf/advika.urdf (robot description, URDF)
Before this commit: robot advika, 12 links, 11 joints
Links:
- added link base_footprint
Joints:
- added joint base_footprint_joint: type fixed, parent base_footprint, child base_link, origin xyz=0 0 0.0 rpy=0 0 0
