Commit message: fix(sim): resolve ros_gz_bridge topic directions and update nav/sim launch configs

File: src/advika_description/urdf/advika.urdf (robot description, URDF)
Before this commit: robot advika, 12 links, 11 joints
Joints:
- joint left_wheel_joint: origin xyz=0 0.115 0.0325 rpy=-1.5708 0 0 -> xyz=0 0.10 0.0325 rpy=-1.5708 0 0
- joint right_wheel_joint: origin xyz=0 -0.115 0.0325 rpy=-1.5708 0 0 -> xyz=0 -0.10 0.0325 rpy=-1.5708 0 0

Commit message: chore: add environment setup and diagnostic reports

File: src/advika_description/urdf/advika.urdf (robot description, URDF)
Before this commit: robot advika, 13 links, 12 joints
Links:
- link base_link: geometry collision box size=0.30 0.24 0.15; visual mesh filename=file:///home/abhishek/Documents/Robotics/advika_robot_ws/si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 scale=0.30 0.24 0.15
